File: rev_a/synchro_power4.kicad_pcb (KiCad board)
At the start: 2 copper layers, 26 parts, among them J1 MB_TERMINATE

Commit message: Rev. A is ready.
Other:
- board outline added: 100 x 100 mm
- rule trace_min: 0.008 -> 0.000315
- rule via_min_size: 0.035 -> 0.001378
- board text added: "(-)7.2V_BAT1(+)"
Changed lines of the file:
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@@
     (links 124)
     (no_connects 0)
-    (area 48.045962 50.149999 152.123372 149.926)
+    (area 48.045962 49.949999 152.123372 150.050001)
     (thickness 1.6)
-    (drawings 21)
+    (drawings 25)
     (tracks 397)
     (zones 0)
@@
     (zone_clearance 0.508)
     (zone_45_only no)
-    (trace_min 0.008)
+    (trace_min 0.000315)
     (segment_width 0.2)
     (edge_width 0.1)
     (via_size 0.889)
     (via_drill 0.635)
-    (via_min_size 0.035)
+    (via_min_size 0.001378)
     (via_min_drill 0.508)
     (uvia_size 0.508)
     (uvia_drill 0.127)
     (uvias_allowed no)
-    (uvia_min_size 0.02)
+    (uvia_min_size 0.000787)
     (uvia_min_drill 0.127)
     (pcb_text_width 0.3)
@@
     (mod_text_size 1 1)
     (mod_text_width 0.15)
-    (pad_size 2.2352 2.2352)
-    (pad_drill 1.016)
+    (pad_size 1.99898 1.99898)
+    (pad_drill 1.00076)
     (pad_to_mask_clearance 0)
     (aux_axis_origin 0 0)
     (visible_elements 7FFEFFFF)
     (pcbplotparams
-      (layerselection 16285697)
+      (layerselection 284721153)
       (usegerberextensions true)
       (excludeedgelayer true)
@@
     )
   )
-  (module Synchro_Power4_Rev_A:RES_10MM (layer F.Cu)
-    (at 99.48 131.86 180)
-    (descr "Resistor, Axial,  RM 10mm, 1/3W,")
-    (tags "Resistor, Axial, RM 10mm, 1/3W,")
-    (fp_text reference R1 (at 7.91 -0.47 180) (layer F.SilkS)
-      (effects (font (size 1.016 1.016) (thickness 0.2032)))
-    )
-    (fp_text value 120 (at 0.02 2.81 180) (layer F.SilkS) hide
-      (effects (font (size 1.016 1.016) (thickness 0.2032)))
-    )
-    (fp_line (start -2.46126 0) (end -3.47726 0) (layer F.SilkS) (width 0.381))
-    (fp_line (start 2.61874 0) (end 3.63474 0) (layer F.SilkS) (width 0.381))
-    (fp_line (start -2.46126 -1.27) (end 2.61874 -1.27) (layer F.SilkS) (width 0.381))
-    (fp_line (start 2.61874 -1.27) (end 2.61874 1.27) (layer F.SilkS) (width 0.381))
-    (fp_line (start 2.61874 1.27) (end -2.46126 1.27) (layer F.SilkS) (width 0.381))
-    (fp_line (start -2.46126 1.27) (end -2.46126 -1.27) (layer F.SilkS) (width 0.381))
-    (pad 1 thru_hole circle (at -5.00126 0 180) (size 1.99898 1.99898) (drill 1.00076) (layers *.Cu)
-      (net 5 "Net-(J1-Pad1)"))
-    (pad 2 thru_hole circle (at 5.15874 0 180) (size 1.99898 1.99898) (drill 1.00076) (layers *.Cu)
-      (net 17 "Net-(N12-Pad16)"))
-  )
   (module Synchro_Power4_Rev_A:TEST_POINT (layer F.Cu)
     (at 68 55)
@@
   (module Synchro_Power4_Rev_A:M5.0_#10_HOLE (layer F.Cu)
     (at 58.57 58.48)
-    (fp_text reference H1 (at 0 0) (layer F.SilkS)
+    (fp_text reference H1 (at 1.48 1.54) (layer F.SilkS)
       (effects (font (size 0.508 0.508) (thickness 0.127)))
     )
@@
       (rotate (xyz 0 0 0))
     )
-  )
-  (module Synchro_Power4_Rev_A:RES_10MM (layer F.Cu)
-    (at 61.02 117.8 180)
-    (descr "Resistor, Axial,  RM 10mm, 1/3W,")
-    (tags "Resistor, Axial, RM 10mm, 1/3W,")
-    (fp_text reference R2 (at -0.03 -2.63 180) (layer F.SilkS)
-      (effects (font (size 1.016 1.016) (thickness 0.2032)))
-    )
-    (fp_text value 120 (at 0.02 2.81 180) (layer F.SilkS) hide
-      (effects (font (size 1.016 1.016) (thickness 0.2032)))
-    )
-    (fp_line (start -2.46126 0) (end -3.47726 0) (layer F.SilkS) (width 0.381))
-    (fp_line (start 2.61874 0) (end 3.63474 0) (layer F.SilkS) (width 0.381))
-    (fp_line (start -2.46126 -1.27) (end 2.61874 -1.27) (layer F.SilkS) (width 0.381))
-    (fp_line (start 2.61874 -1.27) (end 2.61874 1.27) (layer F.SilkS) (width 0.381))
-    (fp_line (start 2.61874 1.27) (end -2.46126 1.27) (layer F.SilkS) (width 0.381))
-    (fp_line (start -2.46126 1.27) (end -2.46126 -1.27) (layer F.SilkS) (width 0.381))
-    (pad 1 thru_hole circle (at -5.00126 0 180) (size 1.99898 1.99898) (drill 1.00076) (layers *.Cu)
-      (net 26 "Net-(R2-Pad1)"))
-    (pad 2 thru_hole circle (at 5.15874 0 180) (size 1.99898 1.99898) (drill 1.00076) (layers *.Cu)
-      (net 27 "Net-(R2-Pad2)"))
   )
   (module Synchro_Power4_Rev_A:TEST_POINT (layer F.Cu)
@@
     )
   )
+  (module Synchro_Power4_Rev_A:RES_10MM (layer F.Cu)
+    (at 61.02 117.8 180)
+    (descr "Resistor, Axial,  RM 10mm, 1/3W,")
+    (tags "Resistor, Axial, RM 10mm, 1/3W,")
+    (fp_text reference R2 (at -0.03 -2.63 180) (layer F.SilkS)
+      (effects (font (size 1.016 1.016) (thickness 0.2032)))
+    )
+    (fp_text value 120 (at 0.02 2.81 180) (layer F.SilkS) hide
+      (effects (font (size 1.016 1.016) (thickness 0.2032)))
+    )
+    (fp_line (start -2.46126 0) (end -3.47726 0) (layer F.SilkS) (width 0.381))
+    (fp_line (start 2.61874 0) (end 3.63474 0) (layer F.SilkS) (width 0.381))
+    (fp_line (start -2.46126 -1.27) (end 2.61874 -1.27) (layer F.SilkS) (width 0.381))
+    (fp_line (start 2.61874 -1.27) (end 2.61874 1.27) (layer F.SilkS) (width 0.381))
+    (fp_line (start 2.61874 1.27) (end -2.46126 1.27) (layer F.SilkS) (width 0.381))
+    (fp_line (start -2.46126 1.27) (end -2.46126 -1.27) (layer F.SilkS) (width 0.381))
+    (pad 1 thru_hole circle (at -5.00126 0 180) (size 1.99898 1.99898) (drill 1.00076) (layers *.Cu *.Mask)
+      (net 26 "Net-(R2-Pad1)"))
+    (pad 2 thru_hole circle (at 5.15874 0 180) (size 1.99898 1.99898) (drill 1.00076) (layers *.Cu *.Mask)
+      (net 27 "Net-(R2-Pad2)"))
+  )
+  (module Synchro_Power4_Rev_A:RES_10MM (layer F.Cu)
+    (at 99.48 131.86 180)
+    (descr "Resistor, Axial,  RM 10mm, 1/3W,")
+    (tags "Resistor, Axial, RM 10mm, 1/3W,")
+    (fp_text reference R1 (at -0.03 -2.63 180) (layer F.SilkS)
+      (effects (font (size 1.016 1.016) (thickness 0.2032)))
+    )
+    (fp_text value 120 (at 0.02 2.81 180) (layer F.SilkS) hide
+      (effects (font (size 1.016 1.016) (thickness 0.2032)))
+    )
+    (fp_line (start -2.46126 0) (end -3.47726 0) (layer F.SilkS) (width 0.381))
+    (fp_line (start 2.61874 0) (end 3.63474 0) (layer F.SilkS) (width 0.381))
+    (fp_line (start -2.46126 -1.27) (end 2.61874 -1.27) (layer F.SilkS) (width 0.381))
+    (fp_line (start 2.61874 -1.27) (end 2.61874 1.27) (layer F.SilkS) (width 0.381))
+    (fp_line (start 2.61874 1.27) (end -2.46126 1.27) (layer F.SilkS) (width 0.381))
+    (fp_line (start -2.46126 1.27) (end -2.46126 -1.27) (layer F.SilkS) (width 0.381))
+    (pad 1 thru_hole circle (at -5.00126 0 180) (size 1.99898 1.99898) (drill 1.00076) (layers *.Cu *.Mask)
+      (net 5 "Net-(J1-Pad1)"))
+    (pad 2 thru_hole circle (at 5.15874 0 180) (size 1.99898 1.99898) (drill 1.00076) (layers *.Cu *.Mask)
+      (net 17 "Net-(N12-Pad16)"))
+  )
+  (gr_line (start 150 50) (end 150 150) (angle 90) (layer Edge.Cuts) (width 0.1))
+  (gr_line (start 50 50) (end 150 50) (angle 90) (layer Edge.Cuts) (width 0.1))
+  (gr_line (start 50 150) (end 50 50) (angle 90) (layer Edge.Cuts) (width 0.1))
+  (gr_line (start 50 150) (end 150 150) (angle 90) (layer Edge.Cuts) (width 0.1))
   (gr_text TERM2 (at 65.99 127.86) (layer F.SilkS)
     (effects (font (size 1.016 1.016) (thickness 0.2032)))
@@
     (effects (font (size 1.016 1.016) (thickness 0.2032)))
   )
-  (gr_text "(-)12V_BAT1(+)" (at 51.69 91.98 270) (layer F.SilkS)
+  (gr_text "(-)7.2V_BAT1(+)" (at 51.69 91.98 270) (layer F.SilkS)
     (effects (font (size 1.016 1.016) (thickness 0.2032)))
   )
@@
   (segment (start 98.79 65.88) (end 98.79 59.94) (width 0.2032) (layer F.Cu) (net 23))
   (segment (start 98.79 59.94) (end 100 58.73) (width 0.2032) (layer F.Cu) (net 23))
-  (segment (start 66.01 125.53) (end 66.01 117.81126) (width 0.2032) (layer F.Cu) (net 26) (status C00000))
-  (segment (start 66.01 117.81126) (end 66.02126 117.8) (width 0.2032) (layer F.Cu) (net 26) (status C00000))
-  (segment (start 55.85 125.53) (end 55.85 117.81126) (width 0.2032) (layer F.Cu) (net 27) (status C00000))
-  (segment (start 55.85 117.81126) (end 55.86126 117.8) (width 0.2032) (layer F.Cu) (net 27) (status C00000))
+  (segment (start 66.01 125.53) (end 66.01 117.81126) (width 0.2032) (layer F.Cu) (net 26))
+  (segment (start 66.01 117.81126) (end 66.02126 117.8) (width 0.2032) (layer F.Cu) (net 26))
+  (segment (start 55.85 125.53) (end 55.85 117.81126) (width 0.2032) (layer F.Cu) (net 27))
+  (segment (start 55.85 117.81126) (end 55.86126 117.8) (width 0.2032) (layer F.Cu) (net 27))
 )
