File: rev_a/synchro_power4.sch (KiCad schematic (older format))
At the start: 26 parts, among them J1 MB_TERMINATE

Commit message: Rev. A is ready.
Connections:
- no-connect marks 4 -> 5
Changed lines of the file:
@@
 Title "Synchro Drive Power"
 Date ""
-Rev ""
+Rev "A"
 Comp ""
 Comment1 ""
@@
 Wire Wire Line
 	5200 6700 5200 6550
+NoConn ~ 8600 4900
 $EndSCHEMATC
